File: eagle/embedded.brd (EAGLE design)
At the start: 74.6 x 77.5 mm, 13 parts, among them T1 2SC1306, T2 2SC1306, T3 2SC1306

Commit message: updated.
Routing:
- net N$15: track 174.7 -> 173.6 mm
Changed lines of the file:
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@@
 <wire x1="46.99" y1="64.77" x2="46.99" y2="54.61" width="0.4064" layer="16"/>
 <via x="46.99" y="54.61" extent="1-16" drill="1"/>
-<wire x1="46.99" y1="54.61" x2="48.26" y2="53.34" width="0.4064" layer="1"/>
-<wire x1="48.26" y1="35.56" x2="46.99" y2="34.29" width="0.4064" layer="1"/>
 <via x="46.99" y="34.29" extent="1-16" drill="1"/>
-<wire x1="48.26" y1="53.34" x2="48.26" y2="35.56" width="0.4064" layer="1"/>
+<wire x1="46.99" y1="54.61" x2="46.99" y2="34.29" width="0.4064" layer="1"/>
 <wire x1="46.99" y1="34.29" x2="46.99" y2="3.81" width="0.4064" layer="16"/>
 <wire x1="46.99" y1="3.81" x2="40.64" y2="-2.54" width="0.4064" layer="16"/>
